File: pins.kicad_sch (KiCad schematic)
At the start: 1 part, among them U1 LFE5U-12F-6BG256C

Commit message: Route flash + jtag resistors
Connections:
- net +2V8: now also U1.F6 (VCCIO0), U1.F7 (VCCIO0); no longer U1.K11 (VCCIO3), U1.L11 (VCCIO3)
- net +3V3: now also U1.K11 (VCCIO3), U1.L11 (VCCIO3); no longer U1.F6 (VCCIO0), U1.F7 (VCCIO0)
Changed lines of the file:
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@@
-    )
-  )
-  (symbol (lib_id "power:+3V3") (at 161.29 31.75 0) (unit 1)
-    (in_bom yes) (on_board yes) (dnp no) (fields_autoplaced)
-    (property "Reference" "#PWR014" (at 161.29 35.56 0)
-      (effects (font (size 1.27 1.27)) hide)
-    )
-    (property "Value" "+3V3" (at 161.29 27.94 0)
-      (effects (font (size 1.27 1.27)))
-    )
-    (property "Footprint" "" (at 161.29 31.75 0)
-      (effects (font (size 1.27 1.27)) hide)
-    )
-    (property "Datasheet" "" (at 161.29 31.75 0)
-      (effects (font (size 1.27 1.27)) hide)
-    )
-    (pin "1")
-    (instances
-      (project "daughterboard"
-        (path "/dce8b7ce-114c-4680-a1bd-14f36a94838a/f7c4c87c-bc57-4b96-a4ee-eca871099c12"
-          (reference "#PWR014") (unit 1)
-        )
-        (path "/dce8b7ce-114c-4680-a1bd-14f36a94838a/f7c4c87c-bc57-4b96-a4ee-eca871099c12/587cd7ec-dd93-49e0-9e25-d509672a562d"
-          (reference "#PWR014") (unit 1)
-        )
-      )
     )
   )
@@
         (path "/dce8b7ce-114c-4680-a1bd-14f36a94838a/f7c4c87c-bc57-4b96-a4ee-eca871099c12/587cd7ec-dd93-49e0-9e25-d509672a562d"
           (reference "#PWR017") (unit 1)
+        )
+      )
+    )
+  )
+  (symbol (lib_id "power:+3V3") (at 168.91 104.14 0) (unit 1)
+    (in_bom yes) (on_board yes) (dnp no) (fields_autoplaced)
+    (property "Reference" "#PWR016" (at 168.91 107.95 0)
+      (effects (font (size 1.27 1.27)) hide)
+    )
+    (property "Value" "+3V3" (at 168.91 100.33 0)
+      (effects (font (size 1.27 1.27)))
+    )
+    (property "Footprint" "" (at 168.91 104.14 0)
+      (effects (font (size 1.27 1.27)) hide)
+    )
+    (property "Datasheet" "" (at 168.91 104.14 0)
+      (effects (font (size 1.27 1.27)) hide)
+    )
+    (pin "1")
+    (instances
+      (project "daughterboard"
+        (path "/dce8b7ce-114c-4680-a1bd-14f36a94838a/f7c4c87c-bc57-4b96-a4ee-eca871099c12"
+          (reference "#PWR016") (unit 1)
+        )
+        (path "/dce8b7ce-114c-4680-a1bd-14f36a94838a/f7c4c87c-bc57-4b96-a4ee-eca871099c12/587cd7ec-dd93-49e0-9e25-d509672a562d"
+          (reference "#PWR019") (unit 1)
         )
       )
@@
     )
   )
+  (symbol (lib_id "power:+2V8") (at 161.29 31.75 0) (unit 1)
+    (in_bom yes) (on_board yes) (dnp no) (fields_autoplaced)
+    (property "Reference" "#PWR028" (at 161.29 35.56 0)
+      (effects (font (size 1.27 1.27)) hide)
+    )
+    (property "Value" "+2V8" (at 161.29 27.94 0)
+      (effects (font (size 1.27 1.27)))
+    )
+    (property "Footprint" "" (at 161.29 31.75 0)
+      (effects (font (size 1.27 1.27)) hide)
+    )
+    (property "Datasheet" "" (at 161.29 31.75 0)
+      (effects (font (size 1.27 1.27)) hide)
+    )
+    (pin "1")
+    (instances
+      (project "daughterboard"
+        (path "/dce8b7ce-114c-4680-a1bd-14f36a94838a/233da297-15ca-4163-a51b-09f27dce3135"
+          (reference "#PWR028") (unit 1)
+        )
+        (path "/dce8b7ce-114c-4680-a1bd-14f36a94838a/f7c4c87c-bc57-4b96-a4ee-eca871099c12/587cd7ec-dd93-49e0-9e25-d509672a562d"
+          (reference "#PWR031") (unit 1)
+        )
+      )
+    )
+  )
   (symbol (lib_id "LFE5U-12F-6BG256C:LFE5U-12F-6BG256C") (at 53.34 54.61 0) (unit 6)
     (in_bom yes) (on_board yes) (dnp no) (fields_autoplaced)
@@
         )
       )
-    )
-  )
-  (symbol (lib_id "power:+2V8") (at 168.91 104.14 0) (unit 1)
-    (in_bom yes) (on_board yes) (dnp no) (fields_autoplaced)
-    (property "Reference" "#PWR019" (at 168.91 107.95 0)
-      (effects (font (size 1.27 1.27)) hide)
-    )
-    (property "Value" "+2V8" (at 168.91 100.33 0)
-      (effects (font (size 1.27 1.27)))
-    )
-    (property "Footprint" "" (at 168.91 104.14 0)
-      (effects (font (size 1.27 1.27)) hide)
-    )
-    (property "Datasheet" "" (at 168.91 104.14 0)
-      (effects (font (size 1.27 1.27)) hide)
-    )
-    (pin "1")
-    (instances
-      (project "daughterboard"
-        (path "/dce8b7ce-114c-4680-a1bd-14f36a94838a/f7c4c87c-bc57-4b96-a4ee-eca871099c12"
-          (reference "#PWR019") (unit 1)
-        )
-        (path "/dce8b7ce-114c-4680-a1bd-14f36a94838a/f7c4c87c-bc57-4b96-a4ee-eca871099c12/587cd7ec-dd93-49e0-9e25-d509672a562d"
-          (reference "#PWR019") (unit 1)
-        )
-      )

Commit message: Route power, FTDI chip
Connections:
- net +2V8 renamed VCCIOB
- net +3V0 renamed VCCIOA
Changed lines of the file:
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@@
-    (stroke (width 0) (type default))
-  )
-  (wire (pts (xy 160.02 33.02) (xy 161.29 33.02))
     (stroke (width 0) (type default))
   )
@@
     (stroke (width 0) (type default))
   )
-  (wire (pts (xy 161.29 33.02) (xy 161.29 31.75))
-    (stroke (width 0) (type default))
-  )
   (wire (pts (xy 264.16 105.41) (xy 262.89 105.41))
     (stroke (width 0) (type default))
@@
     (stroke (width 0) (type default))
   )
-  (wire (pts (xy 262.89 21.59) (xy 262.89 22.86))
-    (stroke (width 0) (type default))
-  )
   (wire (pts (xy 168.91 105.41) (xy 168.91 104.14))
     (stroke (width 0) (type default))
   )
-  (wire (pts (xy 262.89 22.86) (xy 261.62 22.86))
-    (stroke (width 0) (type default))
-  )
   (global_label "R3" (shape input) (at 85.09 127 0) (fields_autoplaced)
     (effects (font (size 1.27 1.27)) (justify left))
@@
     )
   )
+  (global_label "VCCIOA" (shape input) (at 261.62 22.86 0) (fields_autoplaced)
+    (effects (font (size 1.27 1.27)) (justify left))
+    (property "Intersheetrefs" "${INTERSHEET_REFS}" (at 271.1783 22.86 0)
+      (effects (font (size 1.27 1.27)) (justify left) hide)
+    )
+  )
   (global_label "B15" (shape input) (at 201.93 113.03 180) (fields_autoplaced)
     (effects (font (size 1.27 1.27)) (justify right))
@@
     )
   )
+  (global_label "F_MOSI" (shape input) (at 128.27 170.18 0) (fields_autoplaced)
+    (effects (font (size 1.27 1.27)) (justify left))
+    (property "Intersheetrefs" "${INTERSHEET_REFS}" (at 137.8282 170.18 0)
+      (effects (font (size 1.27 1.27)) (justify left) hide)
+    )
+  )
   (global_label "J15" (shape input) (at 262.89 151.13 0) (fields_autoplaced)
     (effects (font (size 1.27 1.27)) (justify left))
@@
     )
   )
+  (global_label "VCCIOB" (shape input) (at 160.02 33.02 0) (fields_autoplaced)
+    (effects (font (size 1.27 1.27)) (justify left))
+    (property "Intersheetrefs" "${INTERSHEET_REFS}" (at 169.7597 33.02 0)
+      (effects (font (size 1.27 1.27)) (justify left) hide)
+    )
+  )
   (global_label "E8" (shape input) (at 261.62 66.04 0) (fields_autoplaced)
     (effects (font (size 1.27 1.27)) (justify left))
@@
     (property "Intersheetrefs" "${INTERSHEET_REFS}" (at 17.6561 64.77 0)
       (effects (font (size 1.27 1.27)) (justify right) hide)
+    )
+  )
+  (global_label "F_MISO" (shape input) (at 128.27 187.96 0) (fields_autoplaced)
+    (effects (font (size 1.27 1.27)) (justify left))
+    (property "Intersheetrefs" "${INTERSHEET_REFS}" (at 137.8282 187.96 0)
+      (effects (font (size 1.27 1.27)) (justify left) hide)
     )
   )
@@
     )
   )
-  (symbol (lib_id "power:+2V8") (at 161.29 31.75 0) (unit 1)
-    (in_bom yes) (on_board yes) (dnp no) (fields_autoplaced)
-    (property "Reference" "#PWR028" (at 161.29 35.56 0)
-      (effects (font (size 1.27 1.27)) hide)
-    )
-    (property "Value" "+2V8" (at 161.29 27.94 0)
-      (effects (font (size 1.27 1.27)))
-    )
-    (property "Footprint" "" (at 161.29 31.75 0)
-      (effects (font (size 1.27 1.27)) hide)
-    )
-    (property "Datasheet" "" (at 161.29 31.75 0)
-      (effects (font (size 1.27 1.27)) hide)
-    )
-    (pin "1")
-    (instances
-      (project "daughterboard"
-        (path "/dce8b7ce-114c-4680-a1bd-14f36a94838a/233da297-15ca-4163-a51b-09f27dce3135"
-          (reference "#PWR028") (unit 1)
-        )
-        (path "/dce8b7ce-114c-4680-a1bd-14f36a94838a/f7c4c87c-bc57-4b96-a4ee-eca871099c12/587cd7ec-dd93-49e0-9e25-d509672a562d"
-          (reference "#PWR031") (unit 1)
-        )
-      )
-    )
-  )
   (symbol (lib_id "LFE5U-12F-6BG256C:LFE5U-12F-6BG256C") (at 53.34 54.61 0) (unit 6)
     (in_bom yes) (on_board yes) (dnp no) (fields_autoplaced)
@@
         )
       )
-    )
-  )
-  (symbol (lib_id "power:+3V0") (at 262.89 21.59 0) (unit 1)
-    (in_bom yes) (on_board yes) (dnp no) (fields_autoplaced)
-    (property "Reference" "#PWR015" (at 262.89 25.4 0)
-      (effects (font (size 1.27 1.27)) hide)
-    )
-    (property "Value" "+3V0" (at 262.89 17.78 0)
-      (effects (font (size 1.27 1.27)))
-    )
-    (property "Footprint" "" (at 262.89 21.59 0)
-      (effects (font (size 1.27 1.27)) hide)
-    )
-    (property "Datasheet" "" (at 262.89 21.59 0)
-      (effects (font (size 1.27 1.27)) hide)
-    )
-    (pin "1")
-    (instances
-      (project "daughterboard"
-        (path "/dce8b7ce-114c-4680-a1bd-14f36a94838a/f7c4c87c-bc57-4b96-a4ee-eca871099c12"
-          (reference "#PWR015") (unit 1)
-        )
-        (path "/dce8b7ce-114c-4680-a1bd-14f36a94838a/f7c4c87c-bc57-4b96-a4ee-eca871099c12/587cd7ec-dd93-49e0-9e25-d509672a562d"
-          (reference "#PWR015") (unit 1)
-        )
-      )
